File: pcb/pcb.kicad_pcb (KiCad board)
At the start: 2 copper layers, 55 x 55 mm, 22 parts, among them J1 LED 1 5V/GND/DIN/DOUT, J2 LED 2 5V/GND/DIN/DOUT, J3 LED 3 5V/GND/DIN/DOUT, J4 LED 4 5V/GND/DIN/DOUT, J5 LED 5 5V/GND/DIN/DOUT, J6 LED 6 5V/GND/DIN/DOUT, J7 LED 7 5V/GND/DIN/DOUT, J8 LED 8 5V/GND/DIN/DOUT, U1 ESP32-C3-SUPER-MINI, U2 74AHCT125

Commit message: update pcb files
Parts:
- added G***: gear_logo, display_parts:gear_logo, F.Cu at (28.8, 43.0)
Connections:
- net /GPIO4 renamed Net-(U1-GPIO4/ADC1/SDA)
Other:
- board text added: "+5V"
- board text added: "DIn"
- board text added: "DOut"
- board text added: "Factorio Lamp LED Display https://github.com/hgschmie/factorio-lamp-led-display Copyright (C) 2026 Henning Schmiedehausen"
- board text added: "GND"
Changed lines of the file:
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@@
 		(capping no)
 		(filling no)
-		(zone_defaults)
 		(grid_origin 20 20)
 		(pcbplotparams
@@
 		(embedded_fonts no)
 	)
+	(footprint "display_parts:gear_logo"
+		(layer "F.Cu")
+		(at 28.75 43)
+		(property "Reference" "G***"
+			(at 0 -7 0)
+			(layer "F.SilkS")
+			(hide yes)
+			(effects
+				(font
+					(size 1 1)
+					(thickness 0.15)
+				)
+			)
+		)
+		(property "Value" "gear_logo"
+			(at 0 7 0)
+			(layer "F.Fab")
+			(effects
+				(font
+					(size 1 1)
+					(thickness 0.15)
+				)
+			)
+		)
+		(property "Datasheet" ""
+			(at 0 0 0)
+			(layer "F.Fab")
+			(hide yes)
+			(effects
+				(font
+					(size 1.27 1.27)
+				)
+			)
+		)
+		(property "Description" ""
+			(at 0 0 0)
+			(layer "F.Fab")
+			(hide yes)
+			(effects
+				(font
+					(size 1.27 1.27)
+				)
+			)
+		)
+		(attr board_only exclude_from_pos_files exclude_from_bom)
+		(duplicate_pad_numbers_are_jumpers no)
+		(fp_poly
+			(pts
+				(xy 0.4137 -5) (xy -0.1773 -5) (xy -0.2555 -4.9806) (xy -0.2998 -4.9291) (xy -0.3816 -4.6532) (xy -0.495 -4.1568)
+				(xy -0.5798 -4.0114) (xy -0.6895 -3.9495) (xy -1.3436 -3.7719) (xy -1.8952 -3.5604) (xy -2.0213 -3.5446)
+				(xy -2.1316 -3.5846) (xy -2.6832 -4.0308) (xy -2.8093 -4.0889) (xy -2.9354 -4.0762) (xy -3.2427 -3.861)
+				(xy -3.6288 -3.4791) (xy -3.6883 -3.3845) (xy -3.6574 -3.2664) (xy -3.2918 -2.6517) (xy -3.23 -2.4705)
+				(xy -3.8434 -1.2096) (xy -3.9064 -1.1168) (xy -3.9914 -1.0659) (xy -4.2435 -1.0229) (xy -4.543 -1.018)
+				(xy -4.8661 -0.9617) (xy -4.9473 -0.8471) (xy -5 -0.5713) (xy -5 0.0985) (xy -4.9806 0.1767) (xy -4.9212 0.224)
+				(xy -4.4878 0.3197) (xy -4.078 0.4368) (xy -4.0205 0.4773) (xy -3.9447 0.6659) (xy -3.8047 1.2018)
+				(xy -3.5507 1.8479) (xy -3.547 1.9583) (xy -3.5943 2.0686) (xy -3.9004 2.431) (xy -4.0877 2.6911)
+				(xy -4.0804 2.8487) (xy -3.9089 3.1075) (xy -3.5264 3.5027) (xy -3.4161 3.5755) (xy -3.3373 3.5791)
+				(xy -3.2506 3.5518) (xy -2.6123 3.1742) (xy -2.431 3.1505) (xy -2.108 3.2961) (xy -1.0048 1.2914)
+				(xy -1.312 0.9969) (xy -1.4745 0.7841) (xy -1.654 0.3034) (xy -1.654 -0.3822) (xy -1.5218 -0.7447)
+				(xy -1.3757 -0.9969) (xy -1.1151 -1.2727) (xy -0.8865 -1.449) (xy -0.7131 -1.5339) (xy -0.3428 -1.654)
+				(xy 0.2797 -1.6503) (xy 0.5792 -1.5467) (xy 0.7526 -1.4587) (xy 1.0205 -1.2806) (xy 1.1502 -1.1544)
+				(xy 1.38 -0.8314) (xy 1.4551 -0.6737) (xy 1.5752 -0.264) (xy 1.58 0.1379) (xy 1.5321 0.398) (xy 1.4679 0.5792)
+				(xy 1.2411 0.9811) (xy 1.0362 1.1896) (xy 0.7447 1.3969) (xy 0.264 1.5752) (xy -0.3428 1.5752) (xy -0.7447 1.443)
+				(xy -1.0048 1.2914) (xy -2.108 3.2961) (xy -1.7928 3.4858) (xy -1.2018 3.7567) (xy -1.1168 3.8258)
+				(xy -1.0659 3.9125) (xy -1.0575 4.1095) (xy -0.9835 4.5193) (xy -0.9792 4.7321) (xy -0.9435 4.8175)
+				(xy -0.8471 4.8776) (xy -0.3428 4.9261) (xy -0.2246 5) (xy -0.1815 4.9939) (xy -0.1064 4.9382) (xy 0.0118 5)
+				(xy 0.0876 4.9963) (xy 0.1343 4.9539) (xy 0.2586 4.6691) (xy 0.3197 4.3302) (xy 0.4361 3.9834) (xy 0.4779 3.924)
+				(xy 0.5713 3.8707) (xy 0.7131 3.8489) (xy 1.2253 3.6931) (xy 1.9109 3.4276) (xy 1.9897 3.4409) (xy 2.1237 3.5264)
+				(xy 2.6378 3.9792) (xy 2.699 4.0107) (xy 2.7856 4.0101) (xy 2.8802 3.9726) (xy 3.2978 3.6507) (xy 3.544 3.4003)
+				(xy 3.5755 3.3373) (xy 3.5791 3.2584) (xy 3.5391 3.1481) (xy 3.1421 2.5099) (xy 3.1118 2.4153) (xy 3.1385 2.3049)
+				(xy 3.4858 1.714) (xy 3.6731 1.249) (xy 3.8058 1.0296) (xy 3.8653 0.9896) (xy 4.0308 0.9466) (xy 4.4248 0.9393)
+				(xy 4.5587 0.9047) (xy 4.7163 0.8974) (xy 4.8109 0.8587) (xy 4.8733 0.7841) (xy 4.8903 0.5082) (xy 4.9315 0.3664)
+				(xy 5 0.264) (xy 5 -0.1852) (xy 4.9782 -0.2301) (xy 4.6927 -0.3422) (xy 4.0386 -0.4822) (xy 3.9453 -0.5355)
+				(xy 3.8974 -0.6107) (xy 3.6537 -1.4224) (xy 3.561 -1.6194) (xy 3.4343 -1.9819) (xy 3.4543 -2.0686)
+				(xy 3.5495 -2.2183) (xy 3.861 -2.5886) (xy 4.0107 -2.8172) (xy 3.9931 -2.9432) (xy 3.7294 -3.2978)
+				(xy 3.3845 -3.6434) (xy 3.2821 -3.6894) (xy 3.1875 -3.6574) (xy 2.5019 -3.2439) (xy 2.3759 -3.2318)
+				(xy 1.7612 -3.5482) (xy 1.1623 -3.8083) (xy 1.0562 -3.8889) (xy 0.9896 -4.0149) (xy 0.8883 -4.88)
+				(xy 0.8471 -4.9139) (xy 0.7131 -4.9521)
+			)
+			(stroke
+				(width 0.01)
+				(type solid)
+			)
+			(fill yes)
+			(layer "F.SilkS")
+		)
+		(embedded_fonts no)
+	)
 	(footprint "Connector_PinHeader_2.54mm:PinHeader_1x04_P2.54mm_Vertical"
 		(layer "F.Cu")
@@
 		(at 71 71)
 		(property "Reference" "H4"
-			(at 0 -4.15 0)
+			(at -5 0.5 0)
 			(unlocked yes)
 			(layer "F.SilkS")
+			(hide yes)
 			(effects
 				(font
@@
 		(at 54.5 30 180)
 		(property "Reference" "C2"
-			(at 2.5 2.5 0)
+			(at 2.5 0 0)
 			(unlocked yes)
 			(layer "F.SilkS")
@@
 			(unlocked yes)
 			(layer "F.SilkS")
+			(hide yes)
 			(effects
 				(font
@@
 		)
 		(fp_text user "U1"
-			(at -3 -4.31 90)
+			(at 0 11.19 90)
 			(unlocked yes)
 			(layer "F.SilkS")
@@
 			)
 		)
-		(fp_text user "Factorio Lamp Driver"
-			(at 8 29.19 90)
+		(fp_text user "U1"
+			(at 0 0.19 90)
 			(unlocked yes)
 			(layer "F.Fab")
@@
 			(layers "*.Cu" "*.Mask")
 			(remove_unused_layers no)
-			(net "/GPIO4")
+			(net "Net-(U1-GPIO4{slash}ADC1{slash}SDA)")
 			(pinfunction "GPIO4/ADC1/SDA_13")
 			(pintype "bidirectional")
@@
 			(unlocked yes)
 			(layer "F.SilkS")
+			(hide yes)
 			(effects
 				(font
@@
 		(at 38 25 -90)
 		(property "Reference" "C1"
-			(at -3 3.5 270)
+			(at 1.5 2.5 270)
 			(unlocked yes)
 			(layer "F.SilkS")
@@
 			(layers "*.Cu" "*.Mask")
 			(remove_unused_layers no)
-			(net "/GPIO4")
+			(net "Net-(U1-GPIO4{slash}ADC1{slash}SDA)")
 			(pinfunction "1_1")
 			(pintype "passive")
@@
 		(at 40.16 54.7 180)
 		(property "Reference" "R1"
-			(at 2.76 -2.3 0)
+			(at 5.16 -0.05 0)
 			(unlocked yes)
 			(layer "F.SilkS")
@@
 			(unlocked yes)
 			(layer "F.SilkS")
+			(hide yes)
 			(effects
 				(font
@@
 		(at 46.88 35.385001)
 		(property "Reference" "U2"
-			(at 3.81 -2.33 0)
+			(at 3.87 -2.635001 0)
 			(unlocked yes)
 			(layer "F.SilkS")
@@
 			(layers "*.Cu" "*.Mask")
 			(remove_unused_layers no)
-			(net "/GPIO4")
+			(net "Net-(U1-GPIO4{slash}ADC1{slash}SDA)")
 			(pintype "input")
 		)
@@
 		(at 24 71)
 		(property "Reference" "H3"
-			(at 0 -4.15 0)
+			(at 4.4 1.5 0)
 			(unlocked yes)
 			(layer "F.SilkS")
+			(hide yes)
 			(effects
 				(font
@@
 		(layer "Edge.Cuts")
 	)
+	(gr_text "Factorio Lamp LED Display\n\nhttps://github.com/hgschmie/factorio-lamp-led-display\nCopyright (C) 2026 Henning Schmiedehausen\n"
+		(at 73 66 90)
+		(layer "F.SilkS")
+		(effects
+			(font
+				(size 0.8 0.8)
+				(thickness 0.125)
+				(bold yes)
+			)
+			(justify left bottom)
+		)
+	)
+	(gr_text "DOut"
+		(at 25.2 67.55 0)
+		(layer "F.SilkS")
+		(effects
+			(font
+				(size 0.8 0.8)
+				(thickness 0.2)
+				(bold yes)
+			)
+			(justify left bottom)
+		)
+	)
+	(gr_text "+5V"
+		(at 25.6 62.5 0)
+		(layer "F.SilkS")
+		(effects
+			(font
+				(size 0.8 0.8)
+				(thickness 0.2)
+				(bold yes)
+			)
+			(justify left bottom)
+		)
+	)
+	(gr_text "GND"
+		(at 25.65 65 0)
+		(layer "F.SilkS")
+		(effects
+			(font
+				(size 0.8 0.8)
+				(thickness 0.2)
+				(bold yes)
+			)
+			(justify left bottom)
+		)
+	)
+	(gr_text "DIn"
+		(at 26.25 60 0)
+		(layer "F.SilkS")
+		(effects
+			(font
+				(size 0.8 0.8)
+				(thickness 0.2)
+				(bold yes)
+			)
+			(justify left bottom)
+		)
+	)
 	(segment
 		(start 62.5 65.12)
@@
 		(width 0.25)
 		(layer "F.Cu")
-		(net "/GPIO4")
+		(net "Net-(U1-GPIO4{slash}ADC1{slash}SDA)")
 	)
 	(segment
@@
 		(width 0.25)
 		(layer "F.Cu")
-		(net "/GPIO4")
+		(net "Net-(U1-GPIO4{slash}ADC1{slash}SDA)")
 	)
 	(segment
@@
 		(width 0.25)
 		(layer "F.Cu")
-		(net "/GPIO4")
+		(net "Net-(U1-GPIO4{slash}ADC1{slash}SDA)")
 	)
 	(segment
@@
 		(width 0.25)
 		(layer "F.Cu")
-		(net "/GPIO4")
+		(net "Net-(U1-GPIO4{slash}ADC1{slash}SDA)")
 	)
 	(segment
